File: Thor_20_romboard/Thor_20_romboard.kicad_sch (KiCad schematic)
At the start: 13 parts, among them J1 EPROM CARD, U1 27128, U2 27128, U3 27256, U4 27256, U5 27256, U6 2764

Commit message: add 3D and good romboard
Connections:
- net A14: now also U3.27 (A14), U4.27 (A14), U5.27 (A14)
- net A15': now also U4.22 (~{OE})
- net NS1: no longer U3.20 (~{CE}), U4.20 (~{CE}), U5.20 (~{CE}), U6.20 (~{CE})
- net NS2: now also U3.20 (~{CE}), U4.20 (~{CE})
- net NS3: now also U5.20 (~{CE}), U6.20 (~{CE})
Changed lines of the file:
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@@
 	(title_block
 		(title "CST Thor  - Clone/Upgrade for Sinclair QL")
-		(date "2025-03-15")
+		(date "2025-03-16")
 		(rev "0,1")
 		(company "(C) 2025 Alvaro Alea Fdz")
@@
 		(comment 2 "CERN Open Hardware Licence Version 2 - Strongly Reciprocal")
 		(comment 3 "Under License")
-		(comment 4 "EXPANSION BOARD")
+		(comment 4 "ROM BOARD")
 	)
 	(junction
@@
 	)
 	(bus_entry
+		(at 290.83 96.52)
+		(size 2.54 2.54)
+		(stroke
+			(width 0)
+			(type default)
+		)
+	)
+	(bus_entry
 		(at 246.38 60.96)
 		(size 2.54 2.54)
@@
 	)
 	(bus_entry
+		(at 335.28 91.44)
+		(size 2.54 2.54)
+		(stroke
+			(width 0)
+			(type default)
+		)
+	)
+	(bus_entry
 		(at 86.36 100.33)
 		(size -2.54 -2.54)
@@
 	)
 	(bus_entry
+		(at 246.38 96.52)
+		(size 2.54 2.54)
+		(stroke
+			(width 0)
+			(type default)
+		)
+	)
+	(bus_entry
 		(at 198.12 68.58)
 		(size -2.54 2.54)
@@
 	)
 	(bus_entry
-		(at 335.28 93.98)
-		(size 2.54 2.54)
-		(stroke
-			(width 0)
-			(type default)
-		)
-	)
-	(bus_entry
 		(at 201.93 88.9)
 		(size 2.54 2.54)
@@
 	)
 	(bus_entry
-		(at 335.28 91.44)
-		(size 2.54 2.54)
-		(stroke
-			(width 0)
-			(type default)
-		)
-	)
-	(bus_entry
 		(at 287.02 63.5)
 		(size -2.54 2.54)
@@
 		)
 	)
+	(bus_entry
+		(at 201.93 96.52)
+		(size 2.54 2.54)
+		(stroke
+			(width 0)
+			(type default)
+		)
+	)
 	(bus
 		(pts
@@
 	(wire
 		(pts
+			(xy 248.92 99.06) (xy 256.54 99.06)
+		)
+		(stroke
+			(width 0)
+			(type default)
+		)
+	)
+	(wire
+		(pts
 			(xy 115.57 63.5) (xy 123.19 63.5)
 		)
@@
 	(wire
 		(pts
-			(xy 243.84 109.22) (xy 255.27 109.22)
+			(xy 245.11 109.22) (xy 256.54 109.22)
 		)
 		(stroke
@@
 		)
 	)
+	(bus
+		(pts
+			(xy 290.83 93.98) (xy 290.83 96.52)
+		)
+		(stroke
+			(width 0)
+			(type default)
+		)
+	)
 	(wire
 		(pts
@@
 		)
 	)
+	(wire
+		(pts
+			(xy 204.47 99.06) (xy 212.09 99.06)
+		)
+		(stroke
+			(width 0)
+			(type default)
+		)
+	)
 	(bus
 		(pts
@@
 		)
 	)
+	(bus
+		(pts
+			(xy 201.93 93.98) (xy 201.93 96.52)
+		)
+		(stroke
+			(width 0)
+			(type default)
+		)
+	)
 	(wire
 		(pts
@@
 		)
 	)
+	(bus
+		(pts
+			(xy 246.38 93.98) (xy 246.38 96.52)
+		)
+		(stroke
+			(width 0)
+			(type default)
+		)
+	)
 	(wire
 		(pts
@@
 	(wire
 		(pts
-			(xy 337.82 96.52) (xy 345.44 96.52)
-		)
-		(stroke
-			(width 0)
-			(type default)
-		)
-	)
-	(wire
-		(pts
 			(xy 248.92 68.58) (xy 256.54 68.58)
 		)
@@
 	(bus
 		(pts
-			(xy 335.28 91.44) (xy 335.28 93.98)
-		)
-		(stroke
-			(width 0)
-			(type default)
-		)
-	)
-	(bus
-		(pts
 			(xy 201.93 88.9) (xy 201.93 91.44)
 		)
@@
 	(wire
 		(pts
+			(xy 293.37 99.06) (xy 300.99 99.06)
+		)
+		(stroke
+			(width 0)
+			(type default)
+		)
+	)
+	(wire
+		(pts
 			(xy 71.12 100.33) (xy 73.66 100.33)
 		)
@@
 		)
 	)
+	(label "A14"
+		(at 295.91 99.06 0)
+		(effects
+			(font
+				(size 1.27 1.27)
+			)
+			(justify left bottom)
+		)
+	)
 	(label "A4"
 		(at 297.18 73.66 0)
@@
 		)
 	)
-	(label "NS1"
+	(label "NS2"
 		(at 248.92 106.68 0)
 		(effects
@@
 	)
 	(label "A15'"
-		(at 247.65 109.22 0)
+		(at 248.92 109.22 0)
 		(effects
 			(font
@@
 		)
 	)
-	(label "NS1"
+	(label "NS3"
 		(at 293.37 106.68 0)
 		(effects
@@
 	)
 	(label "A13"
-		(at 340.36 96.52 0)
+		(at 295.91 96.52 0)
 		(effects
 			(font
@@
 		)
 	)
-	(label "A13"
-		(at 295.91 96.52 0)
+	(label "A10"
+		(at 251.46 88.9 0)
 		(effects
 			(font
@@
 		)
 	)
-	(label "A10"
-		(at 251.46 88.9 0)
+	(label "A14"
+		(at 251.46 99.06 0)
 		(effects
 			(font
@@
 		)
 	)
+	(label "A14"
+		(at 207.01 99.06 0)
+		(effects
+			(font
+				(size 1.27 1.27)
+			)
+			(justify left bottom)
+		)
+	)
 	(label "A3"
 		(at 341.63 71.12 0)
@@
 		)
 	)
-	(label "NS1"
+	(label "NS3"
 		(at 337.82 104.14 0)
 		(effects
@@
 		)
 	)
-	(label "NS1"
+	(label "NS2"
 		(at 204.47 106.68 0)
 		(effects
