File: Thor_20_expansion/Thor_20_expansion.kicad_sch (KiCad schematic)
At the start: 54 parts, among them J1 QL_SLOT_DIN41612_CARD, J2 QL_SLOT_DIN41612_CARD, U1 74LS245, U10 74LS04, U11 74LS05, U2 74LS04, U3 74LS74, U34 74LS04, U35 74LS74, U40 74LS05, U41 74LS03, U42 74LS04, U5 74LS139, U6 74LS04, U7 74LS08, U8 74LS03, U9 74LS113

Commit message: update schematic
Parts:
- removed C10, C11, C12, C13, C14, C15, C16, C17, C18, C19, C20, C21, C22, C23, C24, C25, C26, C27, C28, C29, C30, C31, C32, C33, C34, C43, C44, C45, C46, C47, C52, C58, C59: 100n, Capacitor_THT:C_Disc_D4.3mm_W1.9mm_P5.00mm, symbol Device:C
- removed J1: QL_SLOT_DIN41612_CARD, 8bits:DIN41612_B_2x32_Female_Horizontal_THT, symbol 8bits:QL_SLOT_DIN41612
- removed J2: QL_SLOT_DIN41612_CARD, 8bits:DIN41612_B_2x32_Male_Horizontal_THT, symbol 8bits:QL_SLOT_DIN41612
- removed RN1: 8x150 DIL, Package_DIP:DIP-16_W7.62mm, symbol Device:R_Pack08
- removed RN2, RN3, RN4: 7x1K, Resistor_THT:R_Array_SIP8, symbol Device:R_Network07_Split
- removed U1: 74LS245, Package_DIP:DIP-20_W7.62mm, symbol 74xx:74LS245
- removed U10, U2, U34, U42, U6: 74LS04, Package_DIP:DIP-14_W7.62mm, symbol 74xx:74LS04
- removed U11, U40: 74LS05, Package_DIP:DIP-14_W7.62mm, symbol 74xx:74LS05
- removed U3, U35: 74LS74, Package_DIP:DIP-14_W7.62mm, symbol 74xx:74LS74
- removed U41, U8: 74LS03, Package_DIP:DIP-14_W7.62mm, symbol 74xx:74LS03
- removed U5: 74LS139, Package_DIP:DIP-16_W7.62mm, symbol 74xx:74LS139
- removed U7: 74LS08, Package_DIP:DIP-14_W7.62mm, symbol 74xx:74LS08
- removed U9: 74LS113, Package_DIP:DIP-14_W7.62mm, symbol 74xx:74LS113
Connections:
- no-connect marks 14 -> 0
Other:
- sheet Periferics renamed Printer and Mouse Interfaces
- added sheet Expansion Slots (Slots.kicad_sch)
- added sheet Keyboard and RTC Interface (keyboard.kicad_sch)
- added sheet Power Distribution (power.kicad_sch)
- added sheet SCSI Interface (SCSI.kicad_sch)
