File: Thor_20_expansion/glue.kicad_sch (KiCad schematic)
At the start: 13 parts, among them Q1 MPSA 2369 A, U10 74LS04, U11 74LS05, U2 74LS04, U3 74LS74, U40 74LS05, U5 74LS139, U6 74LS04, U7 74LS08, U8 74LS03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

Commit message: update schematic
Parts:
- removed U11: 74LS05, Package_DIP:DIP-14_W7.62mm, symbol 74xx:74LS05
Connections:
- net ACK_HOLD: now also RN2.8 (R7.2), U40.12, U7.9
Other:
- moved on the sheet: U2A, U2C
Changed lines of the file:
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@@
-	)
-	(junction
-		(at 83.82 60.96)
-		(diameter 0)
-		(color 0 0 0 0)
 	)
 	(junction
@@
 		(color 0 0 0 0)
 	)
+	(junction
+		(at 83.82 45.72)
+		(diameter 0)
+		(color 0 0 0 0)
+	)
 	(no_connect
 		(at 137.16 50.8)
@@
 	(wire
 		(pts
-			(xy 54.61 26.67) (xy 67.31 26.67)
+			(xy 54.61 26.67) (xy 63.5 26.67)
 		)
 		(stroke
@@
 	(wire
 		(pts
-			(xy 106.68 113.03) (xy 102.87 113.03)
-		)
-		(stroke
-			(width 0)
-			(type default)
-		)
-	)
-	(wire
-		(pts
 			(xy 96.52 148.59) (xy 96.52 160.02)
 		)
@@
 	(wire
 		(pts
-			(xy 63.5 60.96) (xy 55.88 60.96)
+			(xy 63.5 45.72) (xy 55.88 45.72)
 		)
 		(stroke
@@
 	(wire
 		(pts
-			(xy 82.55 26.67) (xy 87.63 26.67)
+			(xy 78.74 26.67) (xy 87.63 26.67)
 		)
 		(stroke
@@
 	(wire
 		(pts
-			(xy 106.68 106.68) (xy 106.68 113.03)
+			(xy 106.68 106.68) (xy 106.68 111.76)
 		)
 		(stroke
@@
 	(wire
 		(pts
-			(xy 78.74 60.96) (xy 83.82 60.96)
+			(xy 78.74 45.72) (xy 83.82 45.72)
 		)
 		(stroke
@@
 	(wire
 		(pts
-			(xy 69.85 113.03) (xy 87.63 113.03)
+			(xy 73.66 111.76) (xy 106.68 111.76)
 		)
 		(stroke
@@
 	(label "DS"
 		(at 87.63 60.96 0)
-		(effects
-			(font
-				(size 1.27 1.27)
-			)
-			(justify left bottom)
-		)
-	)
-	(label "E"
-		(at 177.8 49.53 0)
 		(effects
 			(font
@@
 	)
 	(global_label "CS1"
-		(shape input)
+		(shape output)
 		(at 231.14 52.07 0)
 		(fields_autoplaced yes)
@@
 	(global_label "DS'"
 		(shape input)
-		(at 55.88 60.96 180)
+		(at 55.88 45.72 180)
 		(fields_autoplaced yes)
 		(effects
@@
 		)
 		(property "Intersheetrefs" "${INTERSHEET_REFS}"
-			(at 49.8105 60.96 0)
+			(at 49.8105 45.72 0)
 			(effects
 				(font
@@
 	)
 	(global_label "CS2"
-		(shape input)
+		(shape output)
 		(at 231.14 46.99 0)
 		(fields_autoplaced yes)
@@
 	)
 	(global_label "PSEL"
-		(shape input)
+		(shape output)
 		(at 107.95 50.8 0)
 		(fields_autoplaced yes)
@@
 	)
 	(global_label "RTC_AS"
-		(shape input)
+		(shape output)
 		(at 121.92 190.5 0)
 		(fields_autoplaced yes)
@@
 	)
 	(global_label "RAM"
-		(shape input)
+		(shape output)
 		(at 143.51 45.72 0)
 		(fields_autoplaced yes)
@@
 	)
 	(global_label "DS"
-		(shape input)
+		(shape output)
 		(at 93.98 60.96 0)
 		(fields_autoplaced yes)
@@
 	(global_label "ACK_HOLD"
 		(shape input)
-		(at 69.85 113.03 180)
+		(at 73.66 111.76 180)
 		(fields_autoplaced yes)
 		(effects
@@
 		)
 		(property "Intersheetrefs" "${INTERSHEET_REFS}"
-			(at 57.3095 113.03 0)
+			(at 61.1195 111.76 0)
 			(effects
 				(font
@@
 	)
 	(global_label "DTACK"
-		(shape input)
+		(shape output)
 		(at 189.23 90.17 0)
 		(fields_autoplaced yes)
@@
 	)
 	(global_label "68XX"
-		(shape input)
+		(shape output)
 		(at 121.92 162.56 0)
 		(fields_autoplaced yes)
@@
 	)
 	(global_label "QL_DSMC"
-		(shape input)
+		(shape output)
 		(at 186.69 69.85 0)
 		(fields_autoplaced yes)
@@
 	)
 	(global_label "DISC"
-		(shape input)
+		(shape output)
 		(at 121.92 148.59 0)
 		(fields_autoplaced yes)
@@
 	)
 	(global_label "RTC_DS"
-		(shape input)
+		(shape output)
 		(at 121.92 176.53 0)
 		(fields_autoplaced yes)
@@
 	)
 	(global_label "VPA"
-		(shape input)
+		(shape output)
 		(at 255.27 72.39 0)
 		(fields_autoplaced yes)
@@
 				(justify left)
 				(hide yes)
-			)
-		)
-	)
-	(symbol
-		(lib_id "74xx:74LS05")
-		(at 95.25 113.03 0)
-		(unit 3)
-		(exclude_from_sim no)
-		(in_bom yes)
-		(on_board yes)
-		(dnp no)
-		(fields_autoplaced yes)
-		(property "Reference" "U11"
-			(at 95.25 104.14 0)
-			(effects
-				(font
-					(size 1.27 1.27)
-				)
-			)
-		)
-		(property "Value" "74LS05"
-			(at 95.25 106.68 0)
-			(effects
-				(font
-					(size 1.27 1.27)
-				)
-			)
-		)
-		(property "Footprint" "Package_DIP:DIP-14_W7.62mm"
-			(at 95.25 113.03 0)
-			(effects
-				(font
-					(size 1.27 1.27)
-				)
-				(hide yes)
-			)
-		)
-		(property "Datasheet" "http://www.ti.com/lit/gpn/sn74LS05"
-			(at 95.25 113.03 0)
-			(effects
-				(font
-					(size 1.27 1.27)
-				)
-				(hide yes)
-			)
-		)
-		(property "Description" "Inverter Open Collect"
-			(at 95.25 113.03 0)
-			(effects
-				(font
-					(size 1.27 1.27)
-				)
-				(hide yes)
-			)
-		)
-		(pin "11"
-		)
-		(pin "10"
-		)
-		(pin "12"
-		)
-		(pin "13"
-		)
-		(pin "14"
-		)
-		(pin "4"
-		)
-		(pin "3"
-		)
-		(pin "9"
-		)
-		(pin "6"
-		)
-		(pin "5"
-		)
-		(pin "2"
-		)
-		(pin "1"
-		)
-		(pin "8"
-		)
-		(pin "7"
-		)
-		(instances
-			(project "Thor_20_expansion"
-				(path "/6a3b12bb-c660-411d-baf4-d16c05c8b5f5/ee4427c0-a8a6-4267-a821-647dafcb81c6"
-					(reference "U11")
-					(unit 3)
-				)
 			)
 		)
@@
 	(symbol
 		(lib_id "74xx:74LS04")
-		(at 71.12 60.96 0)
+		(at 71.12 45.72 0)
 		(unit 3)
 		(exclude_from_sim no)
@@
 		(dnp no)
 		(property "Reference" "U2"
-			(at 71.12 52.07 0)
+			(at 71.12 36.83 0)
 			(effects
 				(font
@@
 		)
 		(property "Value" "74LS04"
-			(at 71.12 54.61 0)
+			(at 71.12 39.37 0)
 			(effects
 				(font
@@
 		)
 		(property "Footprint" "Package_DIP:DIP-14_W7.62mm"
-			(at 71.12 60.96 0)
+			(at 71.12 45.72 0)
 			(effects
 				(font
@@
 		)
 		(property "Datasheet" "http://www.ti.com/lit/gpn/sn74LS04"
-			(at 71.12 60.96 0)
+			(at 71.12 45.72 0)
 			(effects
 				(font
@@
 		)
 		(property "Description" ""
-			(at 71.12 60.96 0)
+			(at 71.12 45.72 0)
 			(effects
 				(font
@@
 	(symbol
 		(lib_id "74xx:74LS04")
-		(at 74.93 26.67 0)
+		(at 71.12 26.67 0)
 		(unit 1)
 		(exclude_from_sim no)
@@
 		(dnp no)
 		(property "Reference" "U2"
-			(at 74.676 18.034 0)
+			(at 70.866 18.034 0)
 			(effects
 				(font
@@
 		)
 		(property "Value" "74LS04"
-			(at 74.93 20.32 0)
+			(at 71.12 20.32 0)
 			(effects
 				(font
@@
 		)
 		(property "Footprint" "Package_DIP:DIP-14_W7.62mm"
-			(at 74.93 26.67 0)
+			(at 71.12 26.67 0)
 			(effects
 				(font
@@
 		)
 		(property "Datasheet" "http://www.ti.com/lit/gpn/sn74LS04"
-			(at 74.93 26.67 0)
+			(at 71.12 26.67 0)
 			(effects
 				(font
@@
 		)
 		(property "Description" ""
-			(at 74.93 26.67 0)
-			(effects
-				(font
+			(at 71.12 26.67 0)
+			(effects
+				(font
