File: Thor_20_expansion/memory.kicad_sch (KiCad schematic)
At the start: 24 parts, among them J3 EPROM CARD, U14 74LS245, U16 74LS257, U17 74LS257, U18 MB81256, U19 MB81256, U20 MB81256, U21 MB81256, U22 MB81256, U23 MB81256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

Commit message: update schematic
Other:
- moved on the sheet: J3, U14, U16, U17, U18, U19, U20, U21, U22, U23, U24, U25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
