File: Thor_20_expansion/periferic.kicad_sch (KiCad schematic)
At the start: 33 parts, among them J4 Conn_02x13_Counter_Clockwise, J42 DIN-5, J5 DE9_Receptacle_MountingHoles, Q40 MPSA 2369 A, U34 74LS04, U35 74LS74, U36 MC6850, U37 6821, U39 MC146818, U40 74LS05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

Commit message: update schematic
Parts:
- removed BT40: VARTA Mempac, 8bits:BatteryHolder_CST_Thor, symbol Device:Battery_Cell
- removed C2: 4n7, Capacitor_THT:C_Disc_D4.3mm_W1.9mm_P5.00mm, symbol Device:C
- removed C3, C4: 22p, Capacitor_THT:C_Disc_D4.3mm_W1.9mm_P5.00mm, symbol Device:C
- removed C5, C6: 100n, Capacitor_THT:C_Disc_D4.3mm_W1.9mm_P5.00mm, symbol Device:C
- removed C7: 22uF-100uF/16V, Capacitor_THT:CP_Radial_D5.0mm_P2.50mm, symbol Device:C_Polarized
- removed D1, D2: 1N4148, Diode_THT:D_DO-34_SOD68_P10.16mm_Horizontal, symbol Device:D
- removed J42: DIN-5, 8bits:DIN-5-female-pcb-horizontal, symbol Connector:DIN-5
- removed Q40: MPSA 2369 A, Package_TO_SOT_THT:TO-92, symbol Simulation_SPICE:NPN
- removed R3: 150K, Resistor_THT:R_Axial_DIN0207_L6.3mm_D2.5mm_P10.16mm_Horizontal, symbol Device:R
- removed R4: 5M6, Resistor_THT:R_Axial_DIN0207_L6.3mm_D2.5mm_P10.16mm_Horizontal, symbol Device:R
- removed R5: 150, Resistor_THT:R_Axial_DIN0207_L6.3mm_D2.5mm_P10.16mm_Horizontal, symbol Device:R
- removed R6: 1K, Resistor_THT:R_Axial_DIN0207_L6.3mm_D2.5mm_P10.16mm_Horizontal, symbol Device:R
- removed R7, R8: 10K, Resistor_THT:R_Axial_DIN0207_L6.3mm_D2.5mm_P10.16mm_Horizontal, symbol Device:R
- removed RN2: 7x1K, Resistor_THT:R_Array_SIP8, symbol Device:R_Network07_Split
- removed unit 5 of RN4
- removed unit 6 of RN4
- removed U36: MC6850, Package_DIP:DIP-24_W15.24mm, symbol Interface_UART:MC6850
- removed U39: MC146818, Package_DIP:DIP-24_W15.24mm, symbol 8bits:MC146818
- removed U40: 74LS05, Package_DIP:DIP-14_W7.62mm, symbol 74xx:74LS05
- removed unit 1 of U41
- removed unit 2 of U42
- removed unit 3 of U42
- removed U6: 74LS04, Package_DIP:DIP-14_W7.62mm, symbol 74xx:74LS04
- removed U7: 74LS08, Package_DIP:DIP-14_W7.62mm, symbol 74xx:74LS08
- removed Y1: 8Mhz, Crystal:Crystal_HC49-4H_Vertical, symbol Device:Crystal
Connections:
- no-connect marks 12 -> 6
Other:
- moved on the sheet: J4, J5, RN4D, U34A, U34B, U34C, U34D, U34E, U34F, U35A, U35B, U37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
